File: ESP32-C3_breakout.kicad_sch (KiCad schematic)
At the start: 32 parts, among them J1 USB4105-GF-A, J2 Conn_01x11_Male, J3 Conn_01x11_Male, SW1 SW_Push, SW2 SW_Push, U1 LD1117S33TR_SOT223, U2 ESP32-C3, Y1 40MHz

Commit message: Minor improvements
Parts:
- renumbered C10 to C1, C9 to C10, C14 to C11, C13 to C12, C7 to C13, C8 to C14, C11 to C2, C12 to C3, C1 to C4, C2 to C5, C3 to C6, C4 to C7, C5 to C8, C6 to C9, R7 to R2, R6 to R3, R2 to R6, R3 to R7
Other:
- note added: "Power merging"
- note removed: "?"
- moved on the sheet: AE1, C11, C12, C13, C14, D1, L1, R2, R3, U2, Y1

Commit message: General improvements
Parts:
- removed AE1: Antenna, ESP_Antenna:ESPRESSIF_ESP32_MIFA_2.4GHz_Right, symbol Device:Antenna
- removed R2, R3: 22R, Resistor_SMD:R_0603_1608Metric, symbol Device:R
- added AE2: Antenna_Shield, ESP_Antenna:ESPRESSIF_ESP32_MIFA_2.4GHz_Right, symbol Device:Antenna_Shield
- added IC1: STF202-22T1G, Package_SO:TSOP-6_1.65x3.05mm_P0.95mm, symbol STF202-22T1G:STF202-22T1G
- renumbered R4 to R2, R5 to R3, R6 to R4, R7 to R5
Connections:
- net D_N: now also IC1.2 (D(IN)_1)
- net D_P: now also IC1.3 (D(IN)_2)
- net GND: now also AE2.2 (Shield), IC1.6 (GND)
- net USB_+5V: now also IC1.1 (VBUS)
- net USB_D+: now also IC1.4 (D(OUT)_1)
- net USB_D-: now also IC1.5 (D(OUT)_2)
- net at C11.1, L1.2: now also AE2.1 (A)
Other:
- moved on the sheet: J1, R2, R3

Commit message: Power plane improvement
Parts:
- C1: value 10u -> 100n
- C10: renamed from C9; value 0.1u -> 100n
- C6: renamed from C5; value 0.1u -> 100n
- renumbered AE2 to AE1, C10 to C11, C11 to C12, C12 to C13, C13 to C14, C14 to C15, C6 to C7, C7 to C8, C8 to C9
Connections:
- net +3V3: now also J3.10 (Pin_10); no longer J3.2 (Pin_2)
- net EN: now also J3.2 (Pin_2); no longer J3.3 (Pin_3)
- net GND: now also J3.9 (Pin_9), Y1.2, Y1.4; no longer J3.10 (Pin_10), Y1.1, Y1.3
- net GPIO0: now also J3.3 (Pin_3); no longer J3.4 (Pin_4)
- net GPIO1: now also J3.4 (Pin_4); no longer J3.5 (Pin_5)
- net GPIO2: now also J3.5 (Pin_5); no longer J3.6 (Pin_6)
- net GPIO3: now also J3.6 (Pin_6); no longer J3.7 (Pin_7)
- net GPIO4: now also J3.7 (Pin_7); no longer J3.8 (Pin_8)
- net GPIO5: now also J3.8 (Pin_8); no longer J3.9 (Pin_9)
- net at C15.1, U2.30 (XTAL_P): now also Y1.1; no longer Y1.2
- net at C14.1, U2.29 (XTAL_N): now also Y1.3; no longer Y1.4
Other:
- moved on the sheet: Y1

Commit message: General improvements
Parts:
- added C5: 100n, Capacitor_SMD:C_0603_1608Metric, symbol Device:C
Connections:
- net GND: now also C5.2
- net USB_+5V: now also C5.1
Changed lines of the file:
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@@
+    (stroke (width 0) (type default) (color 0 0 0 0))
+  )
+  (wire (pts (xy 105.41 -8.89) (xy 105.41 -7.62))
     (stroke (width 0) (type default) (color 0 0 0 0))
   )
@@
   )
   (polyline (pts (xy 173.99 194.31) (xy 140.97 194.31))
+    (stroke (width 0) (type default) (color 0 0 0 0))
+  )
+  (wire (pts (xy 105.41 -21.59) (xy 105.41 -16.51))
     (stroke (width 0) (type default) (color 0 0 0 0))
   )
@@
     (effects (font (size 1.27 1.27)) (justify left bottom))
   )
+  (label "USB_+5V" (at 105.41 -21.59 180)
+    (effects (font (size 1.27 1.27)) (justify right bottom))
+  )
   (label "GPIO6" (at 212.09 149.86 0)
     (effects (font (size 1.27 1.27)) (justify left bottom))
@@
   )
   (symbol (lib_id "Device:R") (at 83.82 49.53 0) (unit 1)
-    (in_bom yes) (on_board yes) (fields_autoplaced)
+    (in_bom yes) (on_board yes)
     (property "Reference" "R3" (id 0) (at 85.598 48.6953 0)
       (effects (font (size 1.27 1.27)) (justify left))
@@
     )
     (property "Distributor" "https://www.tme.eu/Document/b315665a56acbc42df513c99b390ad98/ROYALOHM-THICKFILM.pdf" (id 4) (at 24.13 48.26 0)
+      (effects (font (size 1.27 1.27)) hide)
+    )
+    (pin "1")
+    (pin "2")
+  )
+  (symbol (lib_id "Device:C") (at 105.41 -12.7 0) (unit 1)
+    (in_bom yes) (on_board yes) (fields_autoplaced)
+    (property "Reference" "C5" (id 0) (at 108.331 -13.5347 0)
+      (effects (font (size 1.27 1.27)) (justify left))
+    )
+    (property "Value" "100n" (id 1) (at 108.331 -10.9978 0)
+      (effects (font (size 1.27 1.27)) (justify left))
+    )
+    (property "Footprint" "Capacitor_SMD:C_0603_1608Metric" (id 2) (at 106.3752 -8.89 0)
+      (effects (font (size 1.27 1.27)) hide)
+    )
+    (property "Datasheet" "https://www.tme.eu/Document/4a42202b32dab16128fe107dd69598cc/samsung-chip-cap.pdf" (id 3) (at 105.41 -12.7 0)
+      (effects (font (size 1.27 1.27)) hide)
+    )
+    (property "Distributor" "https://www.tme.eu/cz/details/cl10a106mq8nnnc/kondenzatory-mlcc-smd-0603/samsung/" (id 4) (at 105.41 -12.7 0)
       (effects (font (size 1.27 1.27)) hide)
     )
@@
     )
     (property "Datasheet" "" (id 3) (at 157.48 38.1 0)
+      (effects (font (size 1.27 1.27)) hide)
+    )
+    (pin "1")
+  )
+  (symbol (lib_id "power:GND") (at 105.41 -7.62 0) (unit 1)
+    (in_bom yes) (on_board yes) (fields_autoplaced)
+    (property "Reference" "#PWR016" (id 0) (at 105.41 -1.27 0)
+      (effects (font (size 1.27 1.27)) hide)
+    )
+    (property "Value" "GND" (id 1) (at 105.41 -3.0575 0))
+    (property "Footprint" "" (id 2) (at 105.41 -7.62 0)
+      (effects (font (size 1.27 1.27)) hide)
+    )
+    (property "Datasheet" "" (id 3) (at 105.41 -7.62 0)
       (effects (font (size 1.27 1.27)) hide)
     )
@@
       (reference "#PWR015") (unit 1) (value "GND") (footprint "")
     )
+    (path "/d5f3a311-1b6a-40c9-aa63-2c65de4ab22a"
+      (reference "#PWR016") (unit 1) (value "GND") (footprint "")
+    )
     (path "/cf6a64b7-5aa1-419b-9d7e-7aa604fbdb36"
       (reference "#PWR017") (unit 1) (value "+3V3") (footprint "")
@@
       (reference "C4") (unit 1) (value "1u") (footprint "Capacitor_SMD:C_0603_1608Metric")
     )
+    (path "/79de331d-9209-43f2-8dda-20a4ad47e9be"
+      (reference "C5") (unit 1) (value "100n") (footprint "Capacitor_SMD:C_0603_1608Metric")
+    )
     (path "/b4a2f3f5-4be6-47e4-a0bd-ddf87cbd66be"
